File: PCB/T9 Keyboard for TESLA meshtastic.kicad_sch (KiCad schematic)
At the start: 27 parts, among them J1 PWR, J2 Spare, SW1 SW_Push, SW10 SW_Push, SW11 SW_Push, SW12 SW_Push, SW2 SW_Push, SW3 SW_Push, SW4 SW_Push, SW5 SW_Push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

Commit message: Finished the PCB.
Parts:
- removed J2: Spare, Connector_PinHeader_2.54mm:PinHeader_1x06_P2.54mm_Vertical, symbol Connector:Conn_01x06_Pin
- added J2: I2C, Connector_PinSocket_2.54mm:PinSocket_1x03_P2.54mm_Vertical, symbol Connector:Conn_01x03_Pin
- SW1, SW10, SW11, SW12, SW2, SW3, SW4, SW5, SW6, SW7, SW8, SW9: footprint (none) -> TESLA:TESLA-3 FK 573 00
Connections:
- net GND: now also J2.3 (Pin_3); no longer A1.4 (GND)
- net SCL: now also J2.2 (Pin_2)
- net SDA: now also J2.1 (Pin_1)
- net column_0: now also A1.6 (D3); no longer A1.15 (D12)
- net column_2: now also A1.15 (D12); no longer A1.13 (D10)
- net row_0: now also A1.5 (D2); no longer A1.2 (D0/RX)
- net row_1: now also A1.7 (D4); no longer A1.1 (D1/TX)
- net row_2: now also A1.8 (D5); no longer A1.5 (D2)
- net row_3: now also A1.13 (D10); no longer A1.6 (D3)
- no-connect marks 12 -> 19
Other:
- note added: "https://chatgpt.com/share/694a6849-bc74-8010-bd0e-4c4d8f2faaa1"
